Commit message: Added chessboard patterns files

File: urdf/kinect.xacro (robot description, xacro)
@@ -6,6 +6,5 @@
   <link name="world"/>
   <joint name="camera_joint" type="fixed">
-    <axis xyz="0 1 0" />
-    <origin xyz="0 0 0.2" rpy="0 0 0"/>
+    <origin xyz="0  0 0.2" rpy="0 0 3.14159"/>
     <parent link="world"/>
     <child link="camera_link"/>

Commit message: removed world from kinect urdf and changed collision model

File: urdf/kinect.xacro (robot description, xacro)
@@ -3,17 +3,10 @@
 <robot name="kinect" xmlns:xacro="http://www.ros.org/wiki/xacro">
   <xacro:include filename="$(find kinect_gazebo)/urdf/kinect.gazebo" />
-  <!-- Used for fixing robot to Gazebo 'base_link' -->
-  <link name="world"/>
-  <joint name="camera_joint" type="fixed">
-    <origin xyz="0  0 0.2" rpy="0 0 3.14159"/>
-    <parent link="world"/>
-    <child link="camera_link"/>
-  </joint>
   <!-- Kinect -->
   <link name="camera_link">
     <collision>
-      <origin xyz="0 0 0" rpy="0 0 0"/>
+      <origin xyz="0 0 0" rpy="0 0 1.5708"/>
       <geometry>
-	    <box size="0.05 0.05 0.05"/>
+	    <mesh filename="package://kinect_gazebo/meshes/kinect.dae"/>
       </geometry>
     </collision>

Commit message: Added frames to urdf and removed from launch

File: urdf/kinect.xacro (robot description, xacro)
@@ -23,3 +23,27 @@
     </inertial>
   </link>
+  <link name="camera_rgb_frame"/>
+  <link name="camera_rgb_optical_frame"/>
+  <link name="camera_depth_frame"/>
+  <link name="camera_depth_optical_frame"/>
+  <joint name="camera_link_to_rgb_frame" type="fixed">
+    <parent link="camera_link"/>
+    <child link="camera_rgb_frame"/>
+    <origin xyz="0 -0.045 0" rpy="0 0 0"/>
+  </joint>
+  <joint name="camera_rgb_to_optical" type="fixed">
+    <parent link="camera_rgb_frame"/>
+    <child link="camera_rgb_optical_frame"/>
+    <origin xyz="0 0 0" rpy="1.5707963267948966 0 1.5707963267948966"/>
+  </joint>
+  <joint name="camera_link_to_depth_frame" type="fixed">
+    <parent link="camera_link"/>
+    <child link="camera_depth_frame"/>
+    <origin xyz="0 -0.02 0" rpy="0 0 0"/>
+  </joint>
+  <joint name="camera_depth_to_optical" type="fixed">
+    <parent link="camera_depth_frame"/>
+    <child link="camera_depth_optical_frame"/>
+    <origin xyz="0 0 0" rpy="1.5707963267948966 0 1.5707963267948966"/>
+  </joint>
 </robot>

Commit message: Sovled problem with urdf tfs and changed minimum range of the sensor

File: urdf/kinect.xacro (robot description, xacro)
@@ -35,5 +35,5 @@
     <parent link="camera_rgb_frame"/>
     <child link="camera_rgb_optical_frame"/>
-    <origin xyz="0 0 0" rpy="1.5707963267948966 0 1.5707963267948966"/>
+    <origin xyz="0 0 0" rpy="-1.5707963267948966 0 -1.5707963267948966"/>
   </joint>
   <joint name="camera_link_to_depth_frame" type="fixed">
@@ -45,5 +45,5 @@
     <parent link="camera_depth_frame"/>
     <child link="camera_depth_optical_frame"/>
-    <origin xyz="0 0 0" rpy="1.5707963267948966 0 1.5707963267948966"/>
+    <origin xyz="0 0 0" rpy="-1.5707963267948966 0 -1.5707963267948966"/>
   </joint>
 </robot>

Commit message: Minor changes

File: urdf/kinect.xacro (robot description, xacro)
@@ -6,5 +6,5 @@
   <link name="camera_link">
     <collision>
-      <origin xyz="0 0 0" rpy="0 0 1.5708"/>
+      <origin xyz="0 -0.005 -0.015" rpy="0 0 1.5708"/>
       <geometry>
 	    <mesh filename="package://kinect_gazebo/meshes/kinect.dae"/>
@@ -12,5 +12,5 @@
     </collision>
     <visual>
-      <origin xyz="0 0 0" rpy="0 0 1.5708"/>
+      <origin xyz="0 -0.005 -0.015" rpy="0 0 1.5708"/>
       <geometry>
 	    <mesh filename="package://kinect_gazebo/meshes/kinect.dae"/>

Commit message: Changed frames to match the simulated camera (all at the same place)

File: urdf/kinect.xacro (robot description, xacro)
@@ -30,5 +30,5 @@
     <parent link="camera_link"/>
     <child link="camera_rgb_frame"/>
-    <origin xyz="0 -0.045 0" rpy="0 0 0"/>
+    <origin xyz="0 0 0" rpy="0 0 0"/>
   </joint>
   <joint name="camera_rgb_to_optical" type="fixed">
@@ -40,5 +40,5 @@
     <parent link="camera_link"/>
     <child link="camera_depth_frame"/>
-    <origin xyz="0 -0.02 0" rpy="0 0 0"/>
+    <origin xyz="0 0 0" rpy="0 0 0"/>
   </joint>
   <joint name="camera_depth_to_optical" type="fixed">
